File: kicad_td/kicad_td/usb.kicad_sch (KiCad schematic)
At the start: 9 parts, among them J1 USB_C_Receptacle_USB2.0_16P, U1 USBLC6-2SC6, U2 XC6206P332MR

Commit message: schematics done
Parts:
- added TP1, TP2, TP3: TestPoint, TestPoint:TestPoint_Pad_D2.0mm, symbol Connector:TestPoint
- C1, C2: JLCPCB Part # (none) -> C52923
- U2: JLCPCB Part # (none) -> C5446
Connections:
- net +3.3V: now also TP3.1
- net +5V: now also TP2.1
- net VBUS: now also TP1.1
