File: kicad_td/kicad_td/kicad_td.kicad_sch (KiCad schematic)
At the start: 0 parts

Commit message: crude placement
Parts:
- added H1, H2, H3, H4: MountingHole_Pad, MountingHole:MountingHole_3.2mm_M3_Pad_Via, symbol Mechanical:MountingHole_Pad
Connections:
- new net GND: H1.1, H2.1, H3.1, H4.1
