File: kicad_td/kicad_td/stm32.kicad_sch (KiCad schematic)
At the start: 17 parts, among them J2 Conn_ST_STDC14, U3 STM32G431KBTx, Y1 16MHz

Commit message: schematics done
Parts:
- C10, C9: JLCPCB Part # (none) -> C32949
- C3, C4, C8: JLCPCB Part # (none) -> C1525
- C5: JLCPCB Part # (none) -> C23733
- C6: JLCPCB Part # (none) -> C15195
- C7: JLCPCB Part # (none) -> C52923
- D1, D2: JLCPCB Part # (none) -> C2286
- J2: JLCPCB Part # (none) -> C3975190
- R3, R4: JLCPCB Part # (none) -> C11702
- U3: JLCPCB Part # (none) -> C529357
Connections:
- no-connect marks 2 -> 17
Changed lines of the file:
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@@
 	)
 	(no_connect
+		(at 111.76 82.55)
+	)
+	(no_connect
 		(at 198.12 68.58)
 	)
+	(no_connect
+		(at 111.76 67.31)
+	)
+	(no_connect
+		(at 86.36 77.47)
+	)
+	(no_connect
+		(at 111.76 80.01)
+	)
+	(no_connect
+		(at 111.76 62.23)
+	)
+	(no_connect
+		(at 111.76 72.39)
+	)
+	(no_connect
+		(at 111.76 77.47)
+	)
+	(no_connect
+		(at 86.36 74.93)
+	)
+	(no_connect
+		(at 86.36 85.09)
+	)
+	(no_connect
+		(at 111.76 74.93)
+	)
+	(no_connect
+		(at 111.76 69.85)
+	)
+	(no_connect
+		(at 111.76 95.25)
+	)
+	(no_connect
+		(at 111.76 59.69)
+	)
+	(no_connect
+		(at 86.36 69.85)
+	)
+	(no_connect
+		(at 111.76 64.77)
+	)
 	(wire
 		(pts
@@
 			)
 		)
+		(property "JLCPCB Part #" "C3975190"
+			(at 210.82 63.5 0)
+			(hide yes)
+			(show_name no)
+			(do_not_autoplace no)
+			(effects
+				(font
+					(size 1.27 1.27)
+				)
+			)
+		)
 		(pin "1"
 		)
@@
 			)
 		)
+		(property "JLCPCB Part #" "C1525"
+			(at 86.36 43.18 0)
+			(hide yes)
+			(show_name no)
+			(do_not_autoplace no)
+			(effects
+				(font
+					(size 1.27 1.27)
+				)
+			)
+		)
 		(pin "1"
 		)
@@
 		(unit 1)
 		(body_style 1)
-		(exclude_from_sim no)
+		(exclude_from_sim yes)
 		(in_bom no)
-		(on_board yes)
-		(in_pos_files yes)
+		(on_board no)
+		(in_pos_files no)
 		(dnp no)
 		(fields_autoplaced yes)
@@
 			)
 		)
+		(property "JLCPCB Part #" "C15195"
+			(at 106.68 43.18 0)
+			(hide yes)
+			(show_name no)
+			(do_not_autoplace no)
+			(effects
+				(font
+					(size 1.27 1.27)
+				)
+			)
+		)
 		(pin "1"
 		)
@@
 			)
 		)
+		(property "JLCPCB Part #" "C52923"
+			(at 115.57 43.18 0)
+			(hide yes)
+			(show_name no)
+			(do_not_autoplace no)
+			(effects
+				(font
+					(size 1.27 1.27)
+				)
+			)
+		)
 		(pin "1"
 		)
@@
 			)
 		)
+		(property "JLCPCB Part #" "C11702"
+			(at 45.72 153.67 0)
+			(hide yes)
+			(show_name no)
+			(do_not_autoplace no)
+			(effects
+				(font
+					(size 1.27 1.27)
+				)
+			)
+		)
 		(pin "2"
 		)
@@
 			)
 		)
+		(property "JLCPCB Part #" "C1525"
+			(at 38.1 60.96 0)
+			(hide yes)
+			(show_name no)
+			(do_not_autoplace no)
+			(effects
+				(font
+					(size 1.27 1.27)
+				)
+			)
+		)
 		(pin "1"
 		)
@@
 		(unit 1)
 		(body_style 1)
-		(exclude_from_sim no)
+		(exclude_from_sim yes)
 		(in_bom no)
-		(on_board yes)
-		(in_pos_files yes)
+		(on_board no)
+		(in_pos_files no)
 		(dnp no)
 		(fields_autoplaced yes)
@@
 			)
 		)
+		(property "JLCPCB Part #" "C529357"
+			(at 99.06 77.47 0)
+			(hide yes)
+			(show_name no)
+			(do_not_autoplace no)
+			(effects
+				(font
+					(size 1.27 1.27)
+				)
+			)
+		)
 		(pin "23"
 		)
@@
 			)
 		)
+		(property "JLCPCB Part #" "C2286"
+			(at 45.72 161.29 90)
+			(hide yes)
+			(show_name no)
+			(do_not_autoplace no)
+			(effects
+				(font
+					(size 1.27 1.27)
+				)
+			)
+		)
 		(pin "1"
 		)
@@
 			)
 		)
+		(property "JLCPCB Part #" "C1525"
+			(at 77.47 43.18 0)
+			(hide yes)
+			(show_name no)
+			(do_not_autoplace no)
+			(effects
+				(font
+					(size 1.27 1.27)
+				)
+			)
+		)
 		(pin "1"
 		)
@@
 			)
 		)
+		(property "JLCPCB Part #" "C11702"
+			(at 60.96 153.67 0)
+			(hide yes)
+			(show_name no)
+			(do_not_autoplace no)
+			(effects
+				(font
+					(size 1.27 1.27)
+				)
+			)
+		)
 		(pin "2"
 		)
@@
 			)
 		)
+		(property "JLCPCB Part #" "C2286"
+			(at 60.96 161.29 90)
+			(hide yes)
+			(show_name no)
+			(do_not_autoplace no)
+			(effects
+				(font
+					(size 1.27 1.27)
+				)
+			)
+		)
 		(pin "1"
 		)
@@
 			)
 		)
+		(property "JLCPCB Part #" "C32949"
+			(at 64.77 71.12 0)
+			(hide yes)
+			(show_name no)
+			(do_not_autoplace no)
+			(effects
+				(font
+					(size 1.27 1.27)
+				)
+			)
+		)
 		(pin "1"
 		)
@@
 			)
 		)
+		(property "JLCPCB Part #" "C23733"
+			(at 68.58 43.18 0)
+			(hide yes)
+			(show_name no)
+			(do_not_autoplace no)
+			(effects
+				(font
+					(size 1.27 1.27)
+				)
+			)
+		)
 		(pin "1"
 		)
@@
 			(hide yes)
 			(show_name no)
+			(do_not_autoplace no)
+			(effects
+				(font
+					(size 1.27 1.27)
+				)
+			)
+		)
+		(property "JLCPCB Part #" "C32949"
+			(at 49.53 71.12 0)
+			(hide yes)
+			(show_name no)

Commit message: crude placement
Connections:
- net STATUS: now also U3.9 (PA4); no longer U3.5 (PA0)
Changed lines of the file:
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@@
 	)
 	(no_connect
-		(at 111.76 67.31)
+		(at 111.76 57.15)
 	)
 	(no_connect
@@
 	(wire
 		(pts
-			(xy 111.76 57.15) (xy 120.65 57.15)
+			(xy 111.76 67.31) (xy 120.65 67.31)
 		)
 		(stroke
@@
 	)
 	(label "STATUS"
-		(at 120.65 57.15 180)
+		(at 120.65 67.31 180)
 		(effects
 			(font

Commit message: fine placement
Connections:
- net STM32_D+: now also U3.22 (PA12); no longer U3.21 (PA11)
- net STM32_D-: now also U3.21 (PA11); no longer U3.22 (PA12)
Changed lines of the file:
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@@
 	(hierarchical_label "STM32_D-"
 		(shape bidirectional)
-		(at 125.73 87.63 0)
+		(at 125.73 85.09 0)
 		(effects
 			(font
@@
 	(hierarchical_label "STM32_D+"
 		(shape bidirectional)
-		(at 125.73 85.09 0)
+		(at 125.73 87.63 0)
 		(effects
 			(font
