File: kicad_td/kicad_td/kicad_td.kicad_pcb (KiCad board)
At the start: 2 copper layers, 50 x 40 mm, 28 parts, among them J1 USB_C_Receptacle_USB2.0_16P, J2 Conn_ST_STDC14, U1 USBLC6-2SC6, U2 XC6206P332MR, U3 STM32G431KBTx, Y1 16MHz

Commit message: fine placement
Parts:
- moved D1 34.4 mm to (97.0, 34.0), turned to -90 degrees
- moved D2 32.8 mm to (94.0, 34.0), turned to -90 degrees
- moved R4 28.1 mm to (97.0, 37.0), turned to 90 degrees
- moved R3 26.2 mm to (94.0, 37.0), turned to 90 degrees
- moved C9 22.3 mm to (103.5, 53.7), turned to -90 degrees
- moved C10 20.4 mm to (100.8, 56.0), turned to 0 degrees
- moved Y1 17.2 mm to (100.8, 53.7), turned to 0 degrees
- moved C5 16.1 mm to (88.6, 44.6)
- moved C3 14.8 mm to (88.6, 45.6)
- moved C7 14.7 mm to (91.4, 43.2), turned to 0 degrees
- moved C6 12.9 mm to (91.4, 44.2), turned to 0 degrees
- moved C4 11.7 mm to (97.4, 54.4), turned to 180 degrees
- moved C8 11.4 mm to (99.3, 50.4), turned to 0 degrees
- moved U3 2.00 mm to (93.0, 50.0), turned to 180 degrees
- moved C1 0.71 mm to (82.7, 37.0)
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Connections:
- U3 pad 21: /STM32/STM32_D+ -> /STM32/STM32_D-
- U3 pad 22: /STM32/STM32_D- -> /STM32/STM32_D+

Commit message: routing + gerber
Routing:
- net /STM32/JTMS/SWDIO: track 0.00 -> 35.6 mm
- net /STM32/JCLK/SWCLK: track 0.00 -> 33.5 mm
- net GND: track 0.00 -> 26.1 mm, vias 0 -> 23
- net /STM32/JTDO/SWO: track 0.00 -> 26.0 mm
- net /STM32/NRST: track 0.00 -> 12.8 mm
- net +3.3V: track 0.00 -> 11.2 mm, vias 0 -> 8
- net /STM32/STATUS: track 0.00 -> 8.81 mm
- net Net-(U3-PF1): track 0.00 -> 7.75 mm
- net /USB/CC1: track 0.00 -> 6.44 mm
- net /STM32/STM32_D-: track 0.00 -> 6.39 mm
- net /USB/CC2: track 0.00 -> 6.11 mm
- net /USB/USB_D-: track 0.00 -> 6.09 mm
- net Net-(U3-PF0): track 0.00 -> 5.90 mm
- net /STM32/STM32_D+: track 0.00 -> 5.79 mm
- net /USB/USB_D+: track 0.00 -> 5.44 mm
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- added copper zone on In2.Cu, net +3.3V
- added copper zone on In2.Cu, net +5V
- added copper zone on B.Cu, net GND
- added copper zone on F.Cu, net GND
- added copper zone on In1.Cu, net GND
- added copper zone on In2.Cu, net VBUS
Other:
- copper layers 2 -> 4
- board text added: "Tuto USB-C 18/09/26 Laurent Fiack Rev 1.0"
